Commit message: added steerign to front wheels

File: src/description/kart_description.urdf (robot description, URDF)
Before this commit: robot ucsd_kart, 2 links, 1 joints
Links:
- added link left_steering_link
- added link right_steering_link

Commit message: changes to driving mechanism of front wheels.

File: src/description/kart_description.urdf (robot description, URDF)
Before this commit: robot ucsd_kart, 4 links, 1 joints
Links:
- removed link left_steering_link
- removed link right_steering_link
- added link steering_link
Joints:
- added joint steering_joint: type revolute, parent base_link, child steering_link, origin xyz=${wheel_xoff} 0 ${-wheel_zoff} rpy=0 0 0, axis 0 0 1, limit lower=-1 upper=1 effort=100 velocity=1

Commit message: added libgazebo_ros_ackermann_drive

File: src/description/kart_description.urdf (robot description, URDF)
Before this commit: robot ucsd_kart, 3 links, 2 joints
Links:
- added link imu_link; collision box size=0.1 0.1 0.1; visual box size=0.1 0.1 0.1
Joints:
- added joint imu_joint: type fixed, parent base_link, child imu_link, origin xyz=${-1*wheel_xoff} 0 ${base_height/2}
