Commit message: raymond

File: src/description/ackermann_test.xacro (robot description, xacro)
@@ -2,4 +2,30 @@
 <robot xmlns:xacro="http://www.ros.org/wiki/xacro" >
     <!-- Back wheel macros -->
+    <xacro:macro name="wheel" params="prefix xpos ypos axle_joint:='base_link' yaw:=0">
+    <link name="${prefix}_wheel_link">
+      <visual>
+        <origin xyz="0 0 0" rpy="${pi/2} 0 ${yaw}"/>
+        <geometry>
+          <cylinder radius="${wheel_radius}" length="${wheel_width}"/>
+        </geometry>
+        <material name="Black">
+          <color rgba="0 0 0 1.0"/>
+        </material>
+      </visual>
+      <collision>
+        <origin xyz="0 0 0" rpy="${pi/2} 0 ${yaw}"/>
+        <geometry>
+          <cylinder radius="${wheel_radius}" length="${wheel_width}"/>
+        </geometry>
+      </collision>
+      <xacro:cylinder_inertia m="50" r="${wheel_radius}" h="${wheel_width}"/>
+    </link>
+    <joint name="${prefix}_wheel_joint" type="continuous">
+      <parent link="${axle_joint if axle_joint is not None else 'base_link'}"/>
+      <child link="${prefix}_wheel_link"/>
+      <origin xyz="${xpos} ${ypos} ${-wheel_radius}" rpy="0 0 0"/>
+      <axis xyz="1 0 0"/>
+    </joint>
+  </xacro:macro>
     <xacro:macro name="wheel" params="prefix x_reflect y_reflect parent_link">
         <link name="${prefix}_link">
@@ -44,40 +70,4 @@
         <origin xyz="${wheel_xoff} 0 ${-wheel_zoff}" rpy="0 0 0"/>
     </joint>
-    <xacro:macro name="wheel_steer" params="prefix x_reflect y_reflect parent_link">
-        <link name="${prefix}_steer_link"/>
-        <joint name="${prefix}_steer_joint" type="revolute">
-            <parent link="${parent_link}"/>
-            <child link="${prefix}_steer_link"/>
-            <axis xyz="0 0 1" rpy="0 0 0" />
-            <limit effort="100" velocity="1" lower="-1" upper="1"/>
-            <origin xyz="0 ${y_reflect*(base_width/2+wheel_ygap)} 0"/>
-        </joint>
-        <link name="${prefix}_wheel_link">
-            <visual>
-                <origin xyz="0 0 0" rpy="${pi/2} 0 0"/>
-                <geometry>
-                    <cylinder radius="${wheel_radius}" length="${wheel_width}"/>
-                </geometry>
-                <material name="Gray">
-                    <color rgba="0.5 0.5 0.5 1.0"/>
-                </material>
-            </visual>
-            <collision>
-                <origin xyz="0 0 0" rpy="${pi/2} 0 0"/>
-                <geometry>
-                  <cylinder radius="${wheel_radius}" length="${wheel_width}"/>
-                </geometry>
-              </collision>
-              <xacro:cylinder_inertia m="0.5" r="${wheel_radius}" h="${wheel_width}"/>
-        </link>
-        <joint name="${prefix}_wheel_joint" type="continuous">
-            <parent link="${prefix}_steer_link"/>
-            <child link="${prefix}_wheel_link"/>
-            <origin xyz="0 0 0" rpy="0 0 0"/>
-            <axis xyz="0 1 0"/>
-        </joint>
-    </xacro:macro>
-    <xacro:wheel_steer prefix="front_left" x_reflect="1" y_reflect="1" parent_link="steering_link"/>
-    <xacro:wheel_steer prefix="front_right" x_reflect="1" y_reflect="-1" parent_link="steering_link"/>
 <gazebo>
     <plugin name="gazebo_ros_ackermann_drive" filename="libgazebo_ros_ackermann_drive.so">
@@ -92,5 +82,5 @@
         <front_right_joint>front_right_wheel_joint</front_right_joint>
         <rear_left_joint>rear_left_joint</rear_left_joint>
-        <rear_right_joint>rear_right_joint</rear_right_joint>
+        <rear_right_joint>rear_right_wheel_joint</rear_right_joint>
         <left_steering_joint>front_left_steer_joint</left_steering_joint>
         <right_steering_joint>front_right_steer_joint</right_steering_joint>
