Commit message: file restructure

File: src/description/ackermann.xacro (robot description, xacro)
@@ -1,28 +1,4 @@
 <?xml version="1.0"?>
-<robot name="ucsd_kart" xmlns:xacro="http://ros.org/wiki/xacro">
-    <!-- Define robot constants -->
-    <xacro:property name="base_width" value="0.31"/>
-    <xacro:property name="base_length" value="1.00"/>
-    <xacro:property name="base_height" value="0.18"/>
-    <xacro:property name="wheel_radius" value="0.10"/>
-    <xacro:property name="wheel_width" value="0.04"/>
-    <xacro:property name="wheel_ygap" value="0.025"/>
-    <xacro:property name="wheel_zoff" value="0.05"/>
-    <xacro:property name="wheel_xoff" value="${base_length/2-0.15}"/>
-    <!-- Define intertial property macros  -->
-    <xacro:macro name="box_inertia" params="m w h d">
-        <inertial>
-        <origin xyz="0 0 0" rpy="${pi/2} 0 ${pi/2}"/>
-        <mass value="${m}"/>
-        <inertia ixx="${(m/12) * (h*h + d*d)}" ixy="0.0" ixz="0.0" iyy="${(m/12) * (w*w + d*d)}" iyz="0.0" izz="${(m/12) * (w*w + h*h)}"/>
-        </inertial>
-    </xacro:macro>
-    <xacro:macro name="cylinder_inertia" params="m r h">
-        <inertial>
-        <origin xyz="0 0 0" rpy="${pi/2} 0 0" />
-        <mass value="${m}"/>
-        <inertia ixx="${(m/12) * (3*r*r + h*h)}" ixy = "0" ixz = "0" iyy="${(m/12) * (3*r*r + h*h)}" iyz = "0" izz="${(m/2) * (r*r)}"/>
-        </inertial>
-    </xacro:macro>
+<robot xmlns:xacro="http://www.ros.org/wiki/xacro" >
     <!-- Robot Base -->
     <link name="base_link">
@@ -126,90 +102,4 @@
     <xacro:wheel_steer prefix="front_left" x_reflect="1" y_reflect="1" parent_link="steering_link"/>
     <xacro:wheel_steer prefix="front_right" x_reflect="1" y_reflect="-1" parent_link="steering_link"/>
-    <link name="imu_link">
-        <visual>
-            <geometry>
-                <box size="0.1 0.1 0.1"/>
-            </geometry>
-        </visual>
-        <collision>
-            <geometry>
-                <box size="0.1 0.1 0.1"/>
-            </geometry>
-        </collision>
-        <xacro:box_inertia m="0.1" w="0.1" d="0.1" h="0.1"/>
-    </link>
-    <joint name="imu_joint" type="fixed">
-        <parent link="base_link"/>
-        <child link="imu_link"/>
-        <origin xyz="${-1*wheel_xoff} 0 ${base_height/2}"/>
-    </joint>
-    <gazebo reference="imu_link">
-        <sensor name="imu_sensor" type="imu">
-            <plugin filename="libgazebo_ros_imu_sensor.so" name="imu_plugin">
-                <ros>
-                    <namespace>/demo</namespace>
-                    <remapping>~/out:=imu</remapping>
-                </ros>
-                <initial_orientation_as_reference>false</initial_orientation_as_reference>
-            </plugin>
-            <always_on>true</always_on>
-            <update_rate>100</update_rate>
-            <visualize>true</visualize>
-            <imu>
-            <angular_velocity>
-                <x>
-                    <noise type="gaussian">
-                        <mean>0.0</mean>
-                        <stddev>2e-4</stddev>
-                        <bias_mean>0.0000075</bias_mean>
-                        <bias_stddev>0.0000008</bias_stddev>
-                    </noise>
-                </x>
-                <y>
-                    <noise type="gaussian">
-                        <mean>0.0</mean>
-                        <stddev>2e-4</stddev>
-                        <bias_mean>0.0000075</bias_mean>
-                        <bias_stddev>0.0000008</bias_stddev>
-                    </noise>
-                </y>
-                <z>
-                    <noise type="gaussian">
-                        <mean>0.0</mean>
-                        <stddev>2e-4</stddev>
-                        <bias_mean>0.0000075</bias_mean>
-                        <bias_stddev>0.0000008</bias_stddev>
-                    </noise>
-                </z>
-            </angular_velocity>
-            <linear_acceleration>
-                <x>
-                    <noise type="gaussian">
-                        <mean>0.0</mean>
-                        <stddev>1.7e-2</stddev>
-                        <bias_mean>0.1</bias_mean>
-                        <bias_stddev>0.001</bias_stddev>
-                    </noise>
-                </x>
-                <y>
-                    <noise type="gaussian">
-                        <mean>0.0</mean>
-                        <stddev>1.7e-2</stddev>
-                        <bias_mean>0.1</bias_mean>
-                        <bias_stddev>0.001</bias_stddev>
-                    </noise>
-                </y>
-                <z>
-                    <noise type="gaussian">
-                        <mean>0.0</mean>
-                        <stddev>1.7e-2</stddev>
-                        <bias_mean>0.1</bias_mean>
-                        <bias_stddev>0.001</bias_stddev>
-                    </noise>
-                </z>
-            </linear_acceleration>
-            </imu>
-        </sensor>
-    </gazebo>
     <plugin name="gazebo_ros_ackermann_drive" filename="libgazebo_ros_ackermann_drive.so">
         <ros>

Commit message: added launch description to use our model with gz

File: src/description/ackermann.xacro (robot description, xacro)
@@ -1,28 +1,4 @@
 <?xml version="1.0"?>
 <robot xmlns:xacro="http://www.ros.org/wiki/xacro" >
-    <!-- Robot Base -->
-    <link name="base_link">
-        <visual>
-            <geometry>
-                <box size="${base_length} ${base_width} ${base_height}"/>
-            </geometry>
-            <material name="Cyan">
-                <color rgba="0 1.0 1.0 1.0"/>
-            </material>
-        </visual>
-        <collision>
-            <geometry>
-              <box size="${base_length} ${base_width} ${base_height}"/>
-            </geometry>
-          </collision>
-          <xacro:box_inertia m="15" w="${base_width}" d="${base_length}" h="${base_height}"/>
-    </link>
-    <!-- Robot Footprint -->
-    <link name="base_footprint"/>
-    <joint name="base_joint" type="fixed">
-        <parent link="base_link"/>
-        <child link="base_footprint"/>
-        <origin xyz="0.0 0.0 ${-(wheel_radius+wheel_zoff)}" rpy="0 0 0"/>
-    </joint>
     <!-- Back wheel macros -->
     <xacro:macro name="wheel" params="prefix x_reflect y_reflect parent_link">

File: src/description/inertia_macros.xacro (robot description, xacro)
@@ -16,3 +16,9 @@
         </inertial>
     </xacro:macro>
+    <xacro:macro name="sphere_inertia" params="m r">
+        <inertial>
+            <mass value="${m}"/>
+            <inertia ixx="${(2/5) * m * (r*r)}" ixy="0.0" ixz="0.0" iyy="${(2/5) * m * (r*r)}" iyz="0.0" izz="${(2/5) * m * (r*r)}"/>
+        </inertial>
+    </xacro:macro>
 </robot>

File: src/description/main.urdf (robot description, URDF)
Before this commit: robot ucsd_kart, 0 links, 0 joints
Links:
- added link base_footprint
- added link base_link; collision box size=${base_length} ${base_width} ${base_height}; visual box size=${base_length} ${base_width} ${base_height}
Joints:
- added joint base_joint: type fixed, parent base_link, child base_footprint, origin xyz=0.0 0.0 ${-(wheel_radius+wheel_zoff)} rpy=0 0 0

Commit message: st1

File: src/description/ackermann.xacro (robot description, xacro)
@@ -42,5 +42,5 @@
         <axis xyz="0 0 1" rpy="0 0 0" />
         <limit effort="100" velocity="1" lower="-1" upper="1"/>
-        <origin xyz="${wheel_xoff} 0 ${-wheel_zoff}" rpy="0 0 0"/>
+        <origin xyz="${wheel_xoff} 0 0" rpy="0 0 0"/>
     </joint>
     <xacro:macro name="wheel_steer" params="prefix x_reflect y_reflect parent_link">
@@ -74,5 +74,5 @@
             <parent link="${prefix}_steer_link"/>
             <child link="${prefix}_wheel_link"/>
-            <origin xyz="0 0 0" rpy="0 0 0"/>
+            <origin xyz="0 0 ${-wheel_zoff}" rpy="0 0 0"/>
             <axis xyz="0 1 0"/>
         </joint>
@@ -80,34 +80,43 @@
     <xacro:wheel_steer prefix="front_left" x_reflect="1" y_reflect="1" parent_link="steering_link"/>
     <xacro:wheel_steer prefix="front_right" x_reflect="1" y_reflect="-1" parent_link="steering_link"/>
-    <plugin name="gazebo_ros_ackermann_drive" filename="libgazebo_ros_ackermann_drive.so">
-        <ros>
-            <namespace>demo</namespace>
-            <remapping>cmd_vel:=cmd_demo</remapping>
-            <remapping>odom:=odom_demo</remapping>
-            <remapping>distance:=distance_demo</remapping>
-        </ros>
-        <update_rate>100.0</update_rate>
-        <front_left_joint>front_left_wheel_joint</front_left_joint>
-        <front_right_joint>front_right_wheel_joint</front_right_joint>
-        <rear_left_joint>rear_left_wheel_joint</rear_left_joint>
-        <rear_right_joint>rear_right_wheel_joint</rear_right_joint>
-        <left_steering_joint>front_left_steer_joint</left_steering_joint>
-        <right_steering_joint>front_right_steer_joint</right_steering_joint>
-        <steering_wheel_joint>steering_joint</steering_wheel_joint>
-        <max_steer>0.6458</max_steer>
-        <max_steering_angle>7.85</max_steering_angle>
-        <max_speed>20</max_speed>
-        <left_steering_pid_gain>1500 0 1</left_steering_pid_gain>
-        <left_steering_i_range>0 0</left_steering_i_range>
-        <right_steering_pid_gain>1500 0 1</right_steering_pid_gain>
-        <right_steering_i_range>0 0</right_steering_i_range>
-        <linear_velocity_pid_gain>1000 0 1</linear_velocity_pid_gain>
-        <linear_velocity_i_range>0 0</linear_velocity_i_range>
-        <publish_odom>true</publish_odom>
-        <publish_odom_tf>true</publish_odom_tf>
-        <publish_wheel_tf>true</publish_wheel_tf>
-        <publish_distance>true</publish_distance>
-        <odometry_frame>odom_demo</odometry_frame>
-        <robot_base_frame>chassis</robot_base_frame>
-    </plugin>
+    <gazebo>
+        <plugin name="gazebo_ros_ackermann_drive" filename="libgazebo_ros_ackermann_drive.so">
+            <ros>
+                <namespace>demo</namespace>
+                <!-- <remapping>cmd_vel:=cmd_demo</remapping>
+                <remapping>odom:=odom_demo</remapping>
+                <remapping>distance:=distance_demo</remapping> -->
+            </ros>
+            <update_rate>100.0</update_rate>
+            <!-- wheels -->
+            <front_left_joint>front_left_wheel_joint</front_left_joint>
+            <front_right_joint>front_right_wheel_joint</front_right_joint>
+            <rear_left_joint>rear_left_wheel_joint</rear_left_joint>
+            <rear_right_joint>rear_right_wheel_joint</rear_right_joint>
+            <left_steering_joint>front_left_steer_joint</left_steering_joint>
+            <right_steering_joint>front_right_steer_joint</right_steering_joint>
+            <steering_wheel_joint>steering_joint</steering_wheel_joint>
+            <!-- Max absolute steer angle for tyre in radians-->
+            <!-- Any cmd_vel angular z greater than this would be capped -->
+            <max_steer>0.6458</max_steer>
+            <!-- Max absolute steering angle of steering wheel -->
+            <max_steering_angle>7.85</max_steering_angle>
+            <!-- Max absolute linear speed in m/s -->
+            <max_speed>20</max_speed>
+            <!-- PID tuning -->
+            <left_steering_pid_gain>1500 0 1</left_steering_pid_gain>
+            <left_steering_i_range>0 0</left_steering_i_range>
+            <right_steering_pid_gain>1500 0 1</right_steering_pid_gain>
+            <right_steering_i_range>0 0</right_steering_i_range>
+            <linear_velocity_pid_gain>1000 0 1</linear_velocity_pid_gain>
+            <linear_velocity_i_range>0 0</linear_velocity_i_range>
+            <!-- output -->
+            <publish_odom>true</publish_odom>
+            <publish_odom_tf>true</publish_odom_tf>
+            <publish_wheel_tf>true</publish_wheel_tf>
+            <publish_distance>true</publish_distance>
+            <odometry_frame>odom_demo</odometry_frame>
+            <robot_base_frame>chassis</robot_base_frame>
+        </plugin>
+    </gazebo>
 </robot>

Commit message: Add interial and collision to kart

File: src/description/ackermann.xacro (robot description, xacro)
@@ -1,7 +1,9 @@
 <?xml version="1.0"?>
 <robot xmlns:xacro="http://www.ros.org/wiki/xacro" >
+  <xacro:property name="steering_bar_radius" value="0.5"/>
+  <xacro:property name="steering_bar_length" value="2.0"/>
     <!-- Back wheel macros -->
     <xacro:macro name="wheel" params="prefix x_reflect y_reflect parent_link">
-        <link name="${prefix}_link">
+        <link name="${prefix}_wheel_link">
             <visual>
                 <origin xyz="0 0 0" rpy="${pi/2} 0 0"/>
@@ -21,19 +23,33 @@
               <xacro:cylinder_inertia m="0.5" r="${wheel_radius}" h="${wheel_width}"/>
         </link>
-        <joint name="${prefix}_joint" type="continuous">
+        <joint name="${prefix}_wheel_joint" type="continuous">
             <parent link="${parent_link}"/>
-            <child link="${prefix}_link"/>
+            <child link="${prefix}_wheel_link"/>
             <origin xyz="${x_reflect*wheel_xoff} ${y_reflect*(base_width/2+wheel_ygap)} ${-wheel_zoff}" rpy="0 0 0"/>
             <axis xyz="0 1 0"/>
+            <limit effort="100" velocity="10"/>
         </joint>
     </xacro:macro>
     <!-- Create back wheels -->
-    <xacro:wheel prefix="rear_left_wheel" x_reflect="-1" y_reflect="1" parent_link="base_link"/>
-    <xacro:wheel prefix="rear_right_wheel" x_reflect="-1" y_reflect="-1" parent_link="base_link"/>
-    <!-- <xacro:wheel prefix="front_left_wheel" x_reflect="1" y_reflect="1" parent_link="base_link"/>
-    <xacro:wheel prefix="front_right_wheel" x_reflect="1" y_reflect="-1" parent_link="base_link"/> -->
+    <xacro:wheel prefix="rear_left" x_reflect="-1" y_reflect="1" parent_link="base_link"/>
+    <xacro:wheel prefix="rear_right" x_reflect="-1" y_reflect="-1" parent_link="base_link"/>
    <!-- FRONT WHEELS -->
    <link name="steering_link">
-        <origin xyz="${wheel_xoff} 0 ${-wheel_zoff}" rpy="0 0 0"/>
+        <visual>
+        <geometry>
+          <cylinder radius="${steering_bar_radius}" length="${steering_bar_length}"/>
+        </geometry>
+        <material name="Black">
+          <color rgba="0 0 0 1.0"/>
+        </material>
+        <origin xyz="$0 0 0" rpy="0 ${pi/2} 0"/>
+      </visual>
+      <collision>
+        <geometry>
+          <cylinder radius="${steering_bar_radius}" length="${steering_bar_length}"/>
+        </geometry>
+        <origin xyz="0 0 0" rpy="0 ${pi/2} 0"/>
+      </collision>
+      <xacro:cylinder_inertia m="0.5" r="${steering_bar_radius}" h="${steering_bar_length}"/>
     </link>
     <joint name="steering_joint" type="revolute">
@@ -41,14 +57,22 @@
         <child link="steering_link"/>
         <axis xyz="0 0 1" rpy="0 0 0" />
-        <limit effort="100" velocity="1" lower="-1" upper="1"/>
+        <limit effort="1" velocity="1" lower="-1" upper="1"/>
         <origin xyz="${wheel_xoff} 0 ${-wheel_zoff}" rpy="0 0 0"/>
     </joint>
     <xacro:macro name="wheel_steer" params="prefix x_reflect y_reflect parent_link">
-        <link name="${prefix}_steer_link"/>
+        <link name="${prefix}_steer_link">
+            <collision>
+                <origin xyz="0 0 0" rpy="${pi/2} 0 0"/>
+                <geometry>
+                  <cylinder radius="${wheel_radius}" length="${wheel_width}"/>
+                </geometry>
+              </collision>
+            <xacro:cylinder_inertia m="0.5" r="${wheel_radius}" h="${wheel_width}"/>
+        </link>
         <joint name="${prefix}_steer_joint" type="revolute">
             <parent link="${parent_link}"/>
             <child link="${prefix}_steer_link"/>
             <axis xyz="0 0 1" rpy="0 0 0" />
-            <limit effort="100" velocity="1" lower="-1" upper="1"/>
+            <limit effort="1" velocity="1" lower="-1" upper="1"/>
             <origin xyz="0 ${y_reflect*(base_width/2+wheel_ygap)} 0"/>
         </joint>
@@ -76,4 +100,5 @@
             <origin xyz="0 0 0" rpy="0 0 0"/>
             <axis xyz="0 1 0"/>
+            <limit effort="100" velocity="10"/>
         </joint>
     </xacro:macro>
@@ -91,12 +116,12 @@
         <front_left_joint>front_left_wheel_joint</front_left_joint>
         <front_right_joint>front_right_wheel_joint</front_right_joint>
-        <rear_left_joint>rear_left_joint</rear_left_joint>
-        <rear_right_joint>rear_right_joint</rear_right_joint>
+        <rear_left_joint>rear_left_wheel_joint</rear_left_joint>
+        <rear_right_joint>rear_right_wheel_joint</rear_right_joint>
         <left_steering_joint>front_left_steer_joint</left_steering_joint>
         <right_steering_joint>front_right_steer_joint</right_steering_joint>
         <steering_wheel_joint>steering_joint</steering_wheel_joint>
         <max_steer>0.6458</max_steer>
-        <max_steering_angle>7.85</max_steering_angle>
-        <max_speed>20</max_speed>
+        <max_steering_angle>0.658</max_steering_angle>
+        <max_speed>1000</max_speed>
         <left_steering_pid_gain>1500 0 1</left_steering_pid_gain>
         <left_steering_i_range>0 0</left_steering_i_range>
