Commit message: added efk with odom + imu

File: src/description/imu_description.xacro (robot description, xacro)
@@ -17,5 +17,5 @@
         <parent link="base_link"/>
         <child link="imu_link"/>
-        <origin xyz="${-1*wheel_xoff} 0 ${base_height/2}"/>
+        <origin xyz="${-1*wheel_xoff} 0 ${base_height/2-.05}"/>
     </joint>
     <gazebo reference="imu_link">
